Commit message: [feature]更新d1h的URDF和mujoco设置

File: urdfs/d1h_description/urdf/robot.urdf (robot description, URDF)
Before this commit: robot d1h_description, 13 links, 12 joints
Links:
- removed link F_docking_link
- removed link F_funtion_link
- added link F_face_link, mass 0.7859; collision box size=0.0495 0.15 0.18; visual mesh filename=package://d1h_description/meshes/face_link.STL
- added link F_locking_link, mass 1.1043; collision box size=0.0495 0.15 0.175; visual mesh filename=package://d1h_description/meshes/locking.STL
- link FL_calf: mass 0.46345045 -> 0.61004; geometry collision box size=0.3 0.04 0.05; visual mesh filename=package://d1h_description/meshes/l_calf.STL
- link FL_foot: mass 1.6631 -> 1.7547; geometry collision cylinder length=0.04 radius=0.087; visual mesh filename=package://d1h_description/meshes/l_foot.STL
- link FL_hip: mass 1.69464273 -> 1.867; geometry visual mesh filename=package://d1h_description/meshes/l_hip.STL
- link FL_thigh: mass 2.55232244 -> 2.8116; geometry collision box size=0.3 0.09 0.05; visual mesh filename=package://d1h_description/meshes/l_thigh.STL
- link FR_calf: mass 0.46345511 -> 0.61004; geometry collision box size=0.3 0.04 0.05; visual mesh filename=package://d1h_description/meshes/r_calf.STL
- link FR_foot: mass 1.6631 -> 1.7547; geometry collision cylinder length=0.04 radius=0.087; visual mesh filename=package://d1h_description/meshes/r_foot.STL
- link FR_hip: mass 1.69464279 -> 1.867; geometry visual mesh filename=package://d1h_description/meshes/r_hip.STL
- link FR_thigh: mass 2.55232278 -> 2.8116; geometry collision box size=0.25 0.09 0.05; visual mesh filename=package://d1h_description/meshes/r_thigh.STL
- link F_base_link: mass 8.44614222 -> 9.158; geometry collision box size=0.275 0.15 0.18; collision box size=0.35 0.15 0.1
- link base_link: mass 0.001 -> None
- link imu_link: mass 0.001 -> None; geometry visual box size=0.001 0.001 0.001
Joints:
- removed joint F_docking_joint
- removed joint F_funtion_joint
- added joint F_face_joint: type fixed, parent F_base_link, child F_face_link, origin xyz=0.1875 0 0 rpy=0 0 0, axis 0 0 0
- added joint F_locking_joint: type fixed, parent F_base_link, child F_locking_link, origin xyz=-0.187 0 0 rpy=0 0 0, axis 0 0 0
- joint FL_calf_joint: axis 0 0 1 -> 0 1 0; limit lower=-2.775 upper=-0.855 effort=80 velocity=20 -> lower=-2.72 upper=-0.85 effort=80 velocity=20; origin xyz=0.25 0 0 rpy=-0.0 0.0 0.0 -> xyz=0 0.091 -0.25 rpy=0 0.85 0
- joint FL_foot_joint: axis 0 0 1 -> 0 1 0; limit lower=-1000000.0 upper=1000000.0 effort=12 velocity=30.0 -> lower=-31415926 upper=31415926 effort=12 velocity=30; origin xyz=0.25 0 0.052166 rpy=0 0 0 -> xyz=0.18376 0.0305 -0.16951 rpy=0 0 0
- joint FL_hip_joint: axis 0 0 1 -> 1 0 0; limit lower=-0.7853981633974483 upper=0.7853981633974483 effort=80 velocity=20 -> lower=-0.7854 upper=0.7854 effort=80 velocity=20; origin xyz=0.0945 0.0775 0 rpy=1.5708 0 1.5708 -> xyz=0.0945 0.0775 0 rpy=0 0 0
- joint FL_thigh_joint: axis 0 0 1 -> 0 1 0; limit lower=-1.8325957145940461 upper=3.4033920413889422 effort=80 velocity=20 -> lower=-1.8326 upper=3.4034 effort=80 velocity=20; origin xyz=0.0905 0 -0.0945 rpy=-1.5708 0 -1.5704 -> xyz=-0.0945 0.0005 0 rpy=0 0 0
- joint FR_calf_joint: axis 0 0 1 -> 0 1 0; limit lower=-2.775 upper=-0.855 effort=80 velocity=20 -> lower=-2.72 upper=-0.85 effort=80 velocity=20; origin xyz=0.25 0 0 rpy=0.0 0.0 0.0 -> xyz=0 -0.091 -0.25 rpy=0 0.85 0
- joint FR_foot_joint: axis 0 0 1 -> 0 1 0; limit lower=-1000000.0 upper=1000000.0 effort=12 velocity=30.0 -> lower=-31415926 upper=31415926 effort=12 velocity=30; origin xyz=0.25 0 -0.052166 rpy=0 0 2.3965 -> xyz=0.18376 -0.0305 -0.16951 rpy=0 0 0
- joint FR_hip_joint: axis 0 0 1 -> 1 0 0; limit lower=-0.7853981633974483 upper=0.7853981633974483 effort=80 velocity=20 -> lower=-0.7854 upper=0.7854 effort=80 velocity=20; origin xyz=0.0945 -0.0775 0 rpy=1.5708 0 1.5708 -> xyz=0.0945 -0.0775 0 rpy=0 0 0
- joint FR_thigh_joint: axis 0 0 1 -> 0 1 0; limit lower=-1.8325957145940461 upper=3.4033920413889422 effort=80 velocity=20 -> lower=-1.8326 upper=3.4034 effort=80 velocity=20; origin xyz=-0.0905 0 -0.0945 rpy=-1.5708 0 -1.5712 -> xyz=-0.0945 -0.0005 0 rpy=0 0 0

File: urdfs/d1h_description/xacro/robot.xacro (robot description, xacro)
@@ -5,6 +5,5 @@
     <xacro:include filename="$(find d1h_description)/xacro/ros2control.xacro"/>
     <xacro:ros2control hw_env="$(arg hw_env)" />
-    <xacro:include filename="$(find d1h_description)/xacro/materials.xacro"/>
-    <xacro:include filename="$(find d1h_description)/xacro/single_robot.xacro"/>
+    <xacro:include filename="$(find d1h_description)/xacro/d1h_base.xacro"/>
     <link name="base_link">
         <visual>
@@ -14,16 +13,6 @@
             </geometry>
         </visual>
-        <inertial>
-            <mass value="0.001"/>
-            <origin rpy="0 0 0" xyz="0 0 0"/>
-            <inertia ixx="0.0001" ixy="0" ixz="0" iyy="0.0001" iyz="0" izz="0.0001"/>
-        </inertial>
     </link>
     <link name="imu_link">
-        <inertial>
-            <mass value="0.001"/>
-            <origin rpy="0 0 0" xyz="0 0 0"/>
-            <inertia ixx="0.0001" ixy="0" ixz="0" iyy="0.0001" iyz="0" izz="0.0001"/>
-        </inertial>
         <visual>
             <origin rpy="0 0 0" xyz="0 0 0"/>
@@ -33,10 +22,4 @@
             <material name="red"/>
         </visual>
-        <collision>
-            <origin rpy="0 0 0" xyz="0 0 0"/>
-            <geometry>
-                <box size=".001 .001 .001"/>
-            </geometry>
-        </collision>
     </link>
     <joint name="imu_joint" type="fixed">
@@ -45,4 +28,4 @@
         <origin rpy="0 0 0" xyz="0 0 0"/>
     </joint>
-    <xacro:single_robot name="F" x_offset="0"/>
+    <xacro:d1h_base name="F" x_offset="0"/>
 </robot>
